Commit message: updated

File: urdf/differential_robot.urdf (robot description, URDF)
Before this commit: robot differential_robot, 4 links, 3 joints
Links:
- added link base_footprint
- added link left_wheel_marker; visual box size=0.03 0.001 0.01
- added link passive_wheel; visual sphere radius=0.005
- added link passive_wheel_holder; visual cylinder length=0.016 radius=0.005
- added link right_wheel_marker; visual box size=0.03 0.001 0.01
- link base_link: geometry visual cylinder length=0.03 radius=0.175
Joints:
- added joint base_to_holder: type fixed, parent base_link, child passive_wheel_holder, origin xyz=0.125 0 -0.023
- added joint footprint_to_base: type fixed, parent base_footprint, child base_link, origin xyz=0 0 0.036
- added joint holder_to_wheel: type fixed, parent passive_wheel_holder, child passive_wheel, origin xyz=0 0 -0.008
- added joint left_wheel_to_marker: type fixed, parent left_wheel, child left_wheel_marker, origin xyz=0 0 0.0155 rpy=-1.57075 0 0
- added joint right_wheel_to_marker: type fixed, parent right_wheel, child right_wheel_marker, origin xyz=0 0 0.0155 rpy=1.57075 0 0
- joint base_to_head: origin xyz=0.125 0 0.066 -> xyz=0.125 0 0.030
- joint base_to_left_wheel: origin xyz=0 0.350 0.036 -> xyz=0 0.175 0 rpy=-1.57075 0 0
- joint base_to_right_wheel: origin xyz=0 -0.350 0.036 -> xyz=0 -0.175 0 rpy=1.57075 0 0

Commit message: added inertia, collision and mass properties

File: urdf/differential_robot.urdf (robot description, URDF)
Before this commit: robot differential_robot, 9 links, 8 joints
Links:
- link base_link: mass None -> 0.100; geometry collision cylinder length=0.03 radius=${basewidth/2}; visual cylinder length=0.03 radius=${basewidth/2}
- link head: mass None -> 0.02; geometry collision box size=0.03 0.03 0.03; visual box size=0.030 0.030 0.030
- link left_wheel: mass None -> ${wheelmass}; geometry collision cylinder length=0.03 radius=${wheelradius}; visual cylinder length=0.03 radius=${wheelradius}
- link passive_wheel: mass None -> 0.02; geometry collision sphere radius=0.005; visual sphere radius=0.005
- link passive_wheel_holder: mass None -> 0.02; geometry collision cylinder length=0.016 radius=0.005; visual cylinder length=0.016 radius=0.005
- link right_wheel: mass None -> ${wheelmass}; geometry collision cylinder length=0.03 radius=${wheelradius}; visual cylinder length=0.030 radius=${wheelradius}
Joints:
- joint base_to_left_wheel: origin xyz=0 0.175 0 rpy=-1.57075 0 0 -> xyz=0 ${basewidth/2} 0 rpy=-1.57075 0 0
- joint base_to_right_wheel: origin xyz=0 -0.175 0 rpy=1.57075 0 0 -> xyz=0 ${-basewidth/2} 0 rpy=1.57075 0 0
