Commit message: Task 8 additions pt 1

File: urdf/differential_robot_simu_task5_part2.urdf (robot description, URDF)
Before this commit: robot differential_robot, 9 links, 8 joints
Links:
- added link laser_connector, mass 0.02; collision cylinder length=0.016 radius=0.005; visual cylinder length=0.016 radius=0.005
- added link laser_emitter, mass 0.015; collision cylinder length=0.030 radius=0.036; visual cylinder length=0.030 radius=0.036
Joints:
- added joint laser_connector_joint: type fixed, parent head, child laser_connector, origin xyz=0 0 0.023 rpy=0 0 0
- added joint laser_emitter_joint: type fixed, parent laser_connector, child laser_emitter, origin xyz=0 0 0.023 rpy=0 0 0
